File: ExtCard/ExtCard.kicad_sch (KiCad schematic)
At the start: 36 parts, among them J1 WIZNET, J3 EXTSPI, Q1 2N3906, Q2 2N3906, Q3 2N3906, U12 MicroSD_SPI_CD, U13 MicroSD_SPI_CD

Commit message: Moved around some traces
Connections:
- net +5V: now also D3.2 (A), D5.2 (A), D7.2 (A); no longer Q1.1 (E), Q2.1 (E), Q3.1 (E)
- net GND: now also R23.2, R30.2, R32.2; no longer D3.1 (K), D5.1 (K), D7.1 (K)
- new net: D7.1 (K), Q1.1 (E)
- new net: D3.1 (K), Q2.1 (E)
- new net: D5.1 (K), Q3.1 (E)
Other:
- moved on the sheet: D3, D5, D7
